Commit message: Add files via upload

File: controlbot_1_description/urdf/controlbot_1.xacro (robot description, xacro)
@@ -76,5 +76,5 @@
   <parent link="base_link"/>
   <child link="wheel_left_link_1"/>
-  <axis xyz="-0.0 1.0 0.0"/>
+  <axis xyz="0.0 1.0 0.0"/>
 </joint>
 <joint name="wheel_right_joint" type="continuous">
@@ -82,5 +82,35 @@
   <parent link="base_link"/>
   <child link="wheel_right_link_1"/>
-  <axis xyz="-0.0 1.0 -0.0"/>
+  <axis xyz="0.0 1.0 0.0"/>
+</joint>
+<link name="imu_link">
+  <inertial>
+    <origin xyz="0.0 0.0 0.0" rpy="0 0 0" />
+    <mass value="0.000528415362211671" />
+    <inertia ixx="1.46176048428261E-08" ixy="0.0" ixz="0.0"
+             iyy="8.59662482954888E-09" iyz="0.0"
+             izz="2.30279421279312E-08" />
+  </inertial>
+  <visual>
+    <origin xyz="0 0 0" rpy="0 0 0" />
+    <geometry>
+      <mesh filename="package://controlbot_1_description/meshes/imu_link.STL" />
+    </geometry>
+    <material name="">
+      <color rgba="0.792156862745098 0.819607843137255 0.933333333333333 1" />
+    </material>
+  </visual>
+  <collision>
+    <origin xyz="0 0 0" rpy="0 0 0" />
+    <geometry>
+      <mesh filename="package://controlbot_1_description/meshes/imu_link.STL" />
+    </geometry>
+  </collision>
+</link>
+<joint name="imu_joint" type="fixed">
+  <origin xyz="0 0 0.027144" rpy="0 0 0" />
+  <parent link="base_link" />
+  <child link="imu_link" />
+  <axis xyz="0 0 0" />
 </joint>
 </robot>

File: controlbot_1_description/urdf/ros2_control.xacro (robot description, xacro)
@@ -11,20 +11,20 @@
             <plugin>gazebo_ros2_control/GazeboSystem</plugin>
         </hardware>
-    <joint name="wheel_right_joint">
+     <joint name="wheel_right_joint">
+         <command_interface name="velocity">
+            <param name="min">-1</param>
+            <param name="max">1</param>
+         </command_interface>
+         <state_interface name="position" />
+         <state_interface name="velocity" />
+     </joint>
+     <joint name="wheel_left_joint">
         <command_interface name="velocity">
-            <param name="min" value="-1"/>
-            <param name="max" value="1"/>
+            <param name="min">-1</param>
+            <param name="max">1</param>
         </command_interface>
-        <state_interface name="position"/>
-        <state_interface name="velocity"/>
-    </joint>
-    <joint name="wheel_left_joint">
-        <command_interface name="velocity">
-            <param name="min" value="-1"/>
-            <param name="max" value="1"/>
-        </command_interface>
-        <state_interface name="position"/>
-        <state_interface name="velocity"/>
-    </joint>
+        <state_interface name="position" />
+        <state_interface name="velocity" />
+     </joint>
     </ros2_control>
 </robot>
