Commit message: Add files via upload

File: controlbot_1_imu_description/urdf/controlbot_1_imu.xacro (robot description, xacro)
@@ -1,4 +1,5 @@
 <?xml version="1.0" ?>
 <robot name="controlbot_1_imu" xmlns:xacro="http://www.ros.org/wiki/xacro">
+<xacro:arg name="is_ignition" default="true"/>
 <xacro:arg name="is_sim" default="true"/>
 <xacro:include filename="$(find controlbot_1_imu_description)/urdf/materials.xacro" />
@@ -6,86 +7,96 @@
 <xacro:include filename="$(find controlbot_1_imu_description)/urdf/controlbot_1_imu.gazebo" />
 <xacro:include filename="$(find controlbot_1_imu_description)/urdf/ros2_control.xacro" />
+<link name="base_footprint"/>
 <link name="base_link">
-  <inertial>
-    <origin xyz="-0.00025879000866563083 6.23198924990529e-05 0.10465970525122006" rpy="0 0 0"/>
-    <mass value="1.1212507191009462"/>
-    <inertia ixx="0.015867" iyy="0.015943" izz="0.014685" ixy="-9e-06" iyz="-2e-06" ixz="0.00016"/>
-  </inertial>
+    <inertial>
+      <origin xyz="0.065 0 -0.056" rpy="0.0 0.25 0.3" />
+      <mass value="1.1172857116478971"/>
+      <inertia ixx="0.013874" iyy="0.013949" izz="0.014621" ixy="-9e-06" iyz="-2e-06" ixz="0.000161"/>
+    </inertial>
   <visual>
-    <origin xyz="0 0 0" rpy="0 0 0"/>
+    <origin xyz="0.065 0 -0.056" rpy="0 0 0"/>
     <geometry>
       <mesh filename="file://$(find controlbot_1_imu_description)/meshes/base_link.stl" scale="0.001 0.001 0.001"/>
     </geometry>
-    <material name="silver"/>
+    <material name="red"/>
   </visual>
   <collision>
-    <origin xyz="0 0 0" rpy="0 0 0"/>
+    <origin xyz="0.065 0 -0.056" rpy="0 0 0"/>
     <geometry>
       <mesh filename="file://$(find controlbot_1_imu_description)/meshes/base_link.stl" scale="0.001 0.001 0.001"/>
     </geometry>
   </collision>
+  <material name="red"/>
 </link>
 <link name="wheel_left_link_1">
-  <inertial>
-    <origin xyz="-1.3877787807814457e-17 0.001539434653235472 -0.0004285178755264324" rpy="0 0 0"/>
-    <mass value="0.16918711951069407"/>
-    <inertia ixx="0.000207" iyy="0.000378" izz="0.000207" ixy="0.0" iyz="-0.0" ixz="0.0"/>
-  </inertial>
+    <inertial>
+      <origin xyz="0.06525 -0.133 -0.056" rpy="0 0 0" />
+      <mass value="0.16918711951069407" />
+      <inertia ixx="0.000207" iyy="0.000378" izz="0.000207" ixy="0.0" iyz="-0.0" ixz="0.0"/>
+    </inertial>
   <visual>
-    <origin xyz="0.065 -0.158849 -0.056855" rpy="0 0 0"/>
+    <origin xyz="0.06525 -0.133 -0.056" rpy="0 0 0"/>
     <geometry>
       <mesh filename="file://$(find controlbot_1_imu_description)/meshes/wheel_left_link_1.stl" scale="0.001 0.001 0.001"/>
     </geometry>
-    <material name="silver"/>
+    <material name="red"/>
   </visual>
   <collision>
-    <origin xyz="0.065 -0.158849 -0.056855" rpy="0 0 0"/>
+    <origin xyz="0.06525 -0.133 -0.056" rpy="0 0 0"/>
     <geometry>
       <mesh filename="file://$(find controlbot_1_imu_description)/meshes/wheel_left_link_1.stl" scale="0.001 0.001 0.001"/>
     </geometry>
+    <material name="red"/>
   </collision>
 </link>
 <link name="wheel_right_link_1">
-  <inertial>
-    <origin xyz="-2.6922908347160046e-15 -0.0016995364726090367 -0.00042637503932518167" rpy="0 0 0"/>
-    <mass value="0.16918711951069396"/>
-    <inertia ixx="0.000207" iyy="0.000378" izz="0.000207" ixy="0.0" iyz="-0.0" ixz="-0.0"/>
-  </inertial>
+    <inertial>
+      <origin xyz="0.06525 0.133 -0.056" rpy="0 0 0" />
+      <mass value="0.16918711951069407" />
+      <inertia ixx="0.000207" iyy="0.000378" izz="0.000207" ixy="0.0" iyz="-0.0" ixz="-0.0"/>
+    </inertial>
   <visual>
-    <origin xyz="0.065 0.15854 -0.056855" rpy="0 0 0"/>
+    <origin xyz="0.06525 0.133 -0.056" rpy="0 0 0"/>
     <geometry>
       <mesh filename="file://$(find controlbot_1_imu_description)/meshes/wheel_right_link_1.stl" scale="0.001 0.001 0.001"/>
     </geometry>
-    <material name="silver"/>
+    <material name="red"/>
   </visual>
   <collision>
-    <origin xyz="0.065 0.15854 -0.056855" rpy="0 0 0"/>
+    <origin xyz="0.06525 0.133 -0.056" rpy="0 0 0"/>
     <geometry>
       <mesh filename="file://$(find controlbot_1_imu_description)/meshes/wheel_right_link_1.stl" scale="0.001 0.001 0.001"/>
     </geometry>
+    <material name="red"/>
   </collision>
 </link>
 <link name="imu_link_1">
-  <inertial>
-    <origin xyz="3.5990916440841465e-06 0.00012513548551613854 0.0016495620864326599" rpy="0 0 0"/>
-    <mass value="0.0019979201495239213"/>
-    <inertia ixx="0.0" iyy="0.0" izz="0.0" ixy="-0.0" iyz="-0.0" ixz="0.0"/>
-  </inertial>
+    <inertial>
+      <origin xyz="0 -0.076 -0.123" rpy="0 0 0" />
+      <mass value="0.0019979201495239213" />
+      <inertia ixx="0.0" iyy="0.0" izz="0.0" ixy="-0.0" iyz="-0.0" ixz="-0.0"/>
+    </inertial>
   <visual>
-    <origin xyz="0.0 -7.4e-05 -0.026572" rpy="0 0 0"/>
+    <origin xyz="0 -0.076 -0.123" rpy="0 0 3.14"/>
     <geometry>
       <mesh filename="file://$(find controlbot_1_imu_description)/meshes/imu_link_1.stl" scale="0.001 0.001 0.001"/>
     </geometry>
-    <material name="silver"/>
+    <material name="red"/>
   </visual>
   <collision>
-    <origin xyz="0.0 -7.4e-05 -0.026572" rpy="0 0 0"/>
+    <origin xyz="0 -0.076 -0.123" rpy="0 0 3.14"/>
     <geometry>
       <mesh filename="file://$(find controlbot_1_imu_description)/meshes/imu_link_1.stl" scale="0.001 0.001 0.001"/>
     </geometry>
+    <material name="red"/>
   </collision>
 </link>
+<joint name="base_joint" type="fixed">
+  <origin xyz="0 0 0.056" rpy="0 0 0"/>
+  <parent link="base_footprint"/>
+  <child link="base_link"/>
+</joint>
 <joint name="wheel_left_joint" type="continuous">
-  <origin xyz="-0.065 0.158849 0.056855" rpy="0 0 0"/>
+  <origin xyz="0 0.133 0" rpy="0 0 0"/>
   <parent link="base_link"/>
   <child link="wheel_left_link_1"/>
@@ -93,5 +104,5 @@
 </joint>
 <joint name="wheel_right_joint" type="continuous">
-  <origin xyz="-0.065 -0.15854 0.056855" rpy="0 0 0"/>
+  <origin xyz="0 -0.133 0" rpy="0 0 0"/>
   <parent link="base_link"/>
   <child link="wheel_right_link_1"/>
@@ -99,5 +110,5 @@
 </joint>
 <joint name="imu_joint" type="fixed">
-  <origin xyz="0.0 7.4e-05 0.026572" rpy="0 0 0"/>
+  <origin xyz="0.065 -0.075 0.06714" rpy="0 0 0"/>
   <parent link="base_link"/>
   <child link="imu_link_1"/>

File: controlbot_1_imu_description/urdf/ros2_control.xacro (robot description, xacro)
@@ -1,17 +1,22 @@
 <?xml version="1.0" ?>
-<robot name="controlbot_1" xmlns:xacro="http://www.ros.org/wiki/xacro">
-    <!--<ros2_control name="RobotSystem" type="system">
-        <xacro:if value="$(arg is_ignition)">
-            <hardware>
-                <plugin>ign_ros2_control/IgnitionSystem</plugin>
-            </hardware>
-        </xacro:if>-->
+<robot name="controlbot_1_imu" xmlns:xacro="http://www.ros.org/wiki/xacro">
     <ros2_control name="RobotSystem" type="system">
+        <!-- ros2_control Gazebo -->
         <xacro:if value="$(arg is_sim)">
-            <hardware>
-                <plugin>gazebo_ros2_control/GazeboSystem</plugin>
-            </hardware>
+            <!-- ROS 2 Humble -->
+            <xacro:if value="$(arg is_ignition)">
+                <hardware>
+                    <plugin>ign_ros2_control/IgnitionSystem</plugin>
+                </hardware>
+            </xacro:if>
+            <!-- ROS 2 Iron or above -->
+            <xacro:unless value="$(arg is_ignition)">
+                <hardware>
+                    <plugin>gz_ros2_control/GazeboSimSystem</plugin>
+                </hardware>
+            </xacro:unless>
         </xacro:if>
-        <xacro:unless>
+        <!-- ros2_control Real Robot -->
+        <xacro:unless value="$(arg is_sim)">
             <hardware>
                 <plugin>controlbot_firmware/controlbotInterface</plugin>

Commit message: Add files via upload

File: controlbot_1_imu_description/urdf/controlbot_1_imu.xacro (robot description, xacro)
@@ -19,5 +19,5 @@
       <mesh filename="file://$(find controlbot_1_imu_description)/meshes/base_link.stl" scale="0.001 0.001 0.001"/>
     </geometry>
-    <material name="red"/>
+    <material name=""/>
   </visual>
   <collision>
@@ -27,5 +27,5 @@
     </geometry>
   </collision>
-  <material name="red"/>
+  <material name=""/>
 </link>
 <link name="wheel_left_link_1">
@@ -40,5 +40,5 @@
       <mesh filename="file://$(find controlbot_1_imu_description)/meshes/wheel_left_link_1.stl" scale="0.001 0.001 0.001"/>
     </geometry>
-    <material name="red"/>
+    <material name=""/>
   </visual>
   <collision>
@@ -47,5 +47,5 @@
       <mesh filename="file://$(find controlbot_1_imu_description)/meshes/wheel_left_link_1.stl" scale="0.001 0.001 0.001"/>
     </geometry>
-    <material name="red"/>
+    <material name=""/>
   </collision>
 </link>
@@ -61,5 +61,5 @@
       <mesh filename="file://$(find controlbot_1_imu_description)/meshes/wheel_right_link_1.stl" scale="0.001 0.001 0.001"/>
     </geometry>
-    <material name="red"/>
+    <material name=""/>
   </visual>
   <collision>
@@ -68,5 +68,5 @@
       <mesh filename="file://$(find controlbot_1_imu_description)/meshes/wheel_right_link_1.stl" scale="0.001 0.001 0.001"/>
     </geometry>
-    <material name="red"/>
+    <material name=""/>
   </collision>
 </link>
@@ -82,5 +82,5 @@
       <mesh filename="file://$(find controlbot_1_imu_description)/meshes/imu_link_1.stl" scale="0.001 0.001 0.001"/>
     </geometry>
-    <material name="red"/>
+    <material name=""/>
   </visual>
   <collision>
@@ -89,5 +89,5 @@
       <mesh filename="file://$(find controlbot_1_imu_description)/meshes/imu_link_1.stl" scale="0.001 0.001 0.001"/>
     </geometry>
-    <material name="red"/>
+    <material name=""/>
   </collision>
 </link>

Commit message: Add files via upload

File: controlbot_1_imu_description/urdf/controlbot_1_imu.xacro (robot description, xacro)
@@ -19,5 +19,5 @@
       <mesh filename="file://$(find controlbot_1_imu_description)/meshes/base_link.stl" scale="0.001 0.001 0.001"/>
     </geometry>
-    <material name=""/>
+    <material name="dark_grey"/>
   </visual>
   <collision>
@@ -40,5 +40,5 @@
       <mesh filename="file://$(find controlbot_1_imu_description)/meshes/wheel_left_link_1.stl" scale="0.001 0.001 0.001"/>
     </geometry>
-    <material name=""/>
+    <material name="black"/>
   </visual>
   <collision>
@@ -61,5 +61,5 @@
       <mesh filename="file://$(find controlbot_1_imu_description)/meshes/wheel_right_link_1.stl" scale="0.001 0.001 0.001"/>
     </geometry>
-    <material name=""/>
+    <material name="black"/>
   </visual>
   <collision>
@@ -73,17 +73,17 @@
 <link name="imu_link_1">
     <inertial>
-      <origin xyz="0 -0.076 -0.123" rpy="0 0 0" />
+      <origin xyz="0 -0.096 -0.123" rpy="0 0 0" />
       <mass value="0.0019979201495239213" />
       <inertia ixx="0.0" iyy="0.0" izz="0.0" ixy="-0.0" iyz="-0.0" ixz="-0.0"/>
     </inertial>
   <visual>
-    <origin xyz="0 -0.076 -0.123" rpy="0 0 3.14"/>
+    <origin xyz="0 -0.096 -0.123" rpy="0 0 3.14"/>
     <geometry>
       <mesh filename="file://$(find controlbot_1_imu_description)/meshes/imu_link_1.stl" scale="0.001 0.001 0.001"/>
     </geometry>
-    <material name=""/>
+    <material name="blue"/>
   </visual>
   <collision>
-    <origin xyz="0 -0.076 -0.123" rpy="0 0 3.14"/>
+    <origin xyz="0 -0.096 -0.123" rpy="0 0 3.14"/>
     <geometry>
       <mesh filename="file://$(find controlbot_1_imu_description)/meshes/imu_link_1.stl" scale="0.001 0.001 0.001"/>
@@ -92,4 +92,26 @@
   </collision>
 </link>
+<link name="laser_link">
+    <inertial>
+      <origin xyz="0 -0.000381929217680526 -0.017064937812947" rpy="0 0 0" />
+      <mass value="0.073084435549317" />
+      <inertia ixx="1.96074931730795E-05" ixy="-3.62091076640009E-07" ixz="4.28230084046735E-07"
+               iyy="2.40983835136327E-05" iyz="1.50180909250652E-08"
+               izz="4.14184164228595E-05" />
+    </inertial>
+    <visual>
+      <origin xyz="0 -0.000381929217680526 -0.017064937812947" rpy="0 0 0" />
+      <geometry>
+        <mesh filename="file://$(find controlbot_1_imu_description)/meshes/laser_link.STL" />
+      </geometry>
+      <material name="black"/>
+    </visual>
+    <collision>
+      <origin xyz="0 -0.000381929217680526 -0.017064937812947" rpy="0 0 0" />
+      <geometry>
+        <mesh filename="file://$(find controlbot_1_imu_description)/meshes/laser_link.STL" />
+      </geometry>
+    </collision>
+  </link>
 <joint name="base_joint" type="fixed">
   <origin xyz="0 0 0.056" rpy="0 0 0"/>
@@ -110,7 +132,13 @@
 </joint>
 <joint name="imu_joint" type="fixed">
-  <origin xyz="0.065 -0.075 0.06714" rpy="0 0 0"/>
+  <origin xyz="0.065 -0.095 0.06714" rpy="0 0 0"/>
   <parent link="base_link"/>
   <child link="imu_link_1"/>
 </joint>
+<joint name="laser_joint" type="fixed">
+    <origin xyz="0.065 0 0.246144" rpy="0 0 3.14" />
+    <parent link="base_link" />
+    <child link="laser_link" />
+    <axis xyz="0 0 0" />
+  </joint>
 </robot>

File: controlbot_1_imu_description/urdf/materials.xacro (robot description, xacro)
@@ -1,6 +1,18 @@
 <?xml version="1.0" ?>
 <robot name="controlbot_1_imu" xmlns:xacro="http://www.ros.org/wiki/xacro" >
+<!--<material name="silver">
+  <color rgba="0.700 0.700 0.700 1.000"/>
+</material>-->
+<material name="blue">
+  <color rgba="0 0 1 1"/>
+</material>
+<material name="black">
+  <color rgba="0 0 0 1"/>
+</material>
 <material name="silver">
-  <color rgba="0.700 0.700 0.700 1.000"/>
+  <color rgba="0.79 0.82 0.93 1"/>
+</material>
+<material name="dark_grey">
+  <color rgba="0.3 0.3 0.3 1"/>
 </material>
 </robot>

File: controlbot_1_imu_description/urdf/ros2_control.xacro (robot description, xacro)
@@ -20,6 +20,6 @@
         <xacro:unless value="$(arg is_sim)">
             <hardware>
-                <plugin>controlbot_firmware/controlbotInterface</plugin>
-                <param name="port">/dev/ttyACM0</param>
+                <plugin>controlbot_firmware/ControlbotInterface</plugin>
+                <param name="port">/dev/ttyUSB0</param>
             </hardware>
         </xacro:unless>

Commit message: Add files via upload

File: controlbot_1_imu_description/urdf/controlbot_1_imu.xacro (robot description, xacro)
@@ -137,5 +137,5 @@
 </joint>
 <joint name="laser_joint" type="fixed">
-    <origin xyz="0.065 0 0.246144" rpy="0 0 3.14" />
+    <origin xyz="0.065 0 0.246144" rpy="0 0 0" />
     <parent link="base_link" />
     <child link="laser_link" />

Commit message: Add files via upload

File: controlbot_1_imu_description/urdf/controlbot_1_imu.xacro (robot description, xacro)
@@ -137,5 +137,5 @@
 </joint>
 <joint name="laser_joint" type="fixed">
-    <origin xyz="0.065 0 0.246144" rpy="0 0 0" />
+    <origin xyz="0.065 0 0.246144" rpy="0 0 3.14" />
     <parent link="base_link" />
     <child link="laser_link" />
